File: Project 3 - MCU Datalogger.kicad_sch (KiCad schematic)
At the start: 0 parts

Commit message: Added symbols to schema (forgot to do this last time)
Parts:
- added BT1: Battery, symbol Device:Battery
- added C1, C2, C3, C4: C, symbol Device:C
- added C5: C_Polarized, symbol Device:C_Polarized
- added D1, D2: LED, symbol Device:LED
- added H1, H2, H3, H4: MountingHole, symbol Mechanical:MountingHole
- added R1, R2, R3, R4, R5, R6, R7: R, symbol Device:R
- added U1, U2: 24LC1025, symbol Memory_EEPROM:24LC1025
- added U3: ATMEGA328P-AU, digikey-footprints:TQFP-32_7x7mm, symbol dk_Embedded-Microcontrollers:ATMEGA328P-AU
- added U4: DS1337S+, SOIC127P600X175-8N, symbol DS1337S_:DS1337S+
- added Y1, Y2: Crystal, symbol Device:Crystal
Other:
- added sheet Connectors (connectors.kicad_sch)
